Commit message: good values in urdf (chassis and wheels)

File: humble/workspace/src/my_bot/description/robot_core.xacro (robot description, xacro)
@@ -1,5 +1,4 @@
 <?xml version="1.0"?>
 <robot xmlns:xacro="http://www.ros.org/wiki/xacro" >
-    <xacro:include filename="inertial_macros.xacro"/>
     <material name="white">
         <color rgba="1 1 1 1" />
@@ -21,23 +20,14 @@
         <parent link="base_link"/>
         <child link="chassis"/>
-        <origin xyz="-0.1 0 0"/>
+        <origin xyz="-0.055 0 0"/>
     </joint>
     <link name="chassis">
         <visual>
-            <origin xyz="0.15 0 0.075"/>
+            <origin xyz="0.1025 0 0.0425"/>
             <geometry>
-                <box size="0.3 0.3 0.15"/>
+                <box size="0.205 0.125 0.085"/>
             </geometry>
             <material name="white"/>
         </visual>
-        <collision>
-            <origin xyz="0.15 0 0.075"/>
-            <geometry>
-                <box size="0.3 0.3 0.15"/>
-            </geometry>
-        </collision>
-        <xacro:inertial_box mass="0.5" x="0.3" y="0.3" z="0.15">
-            <origin xyz="0.15 0 0.075" rpy="0 0 0"/>
-        </xacro:inertial_box>
     </link>
     <!-- LEFT WHEEL LINK -->
@@ -45,5 +35,5 @@
         <parent link="base_link"/>
         <child link="left_wheel"/>
-        <origin xyz="0 0.175 0" rpy="-${pi/2} 0 0" />
+        <origin xyz="0 0.080 0" rpy="-${pi/2} 0 0" />
         <axis xyz="0 0 1"/>
     </joint>
@@ -51,22 +41,14 @@
         <visual>
             <geometry>
-                <cylinder radius="0.05" length="0.04"/>
+                <cylinder radius="0.033" length="0.027"/>
             </geometry>
             <material name="blue"/>
         </visual>
-        <collision>
-            <geometry>
-                <cylinder radius="0.05" length="0.04"/>
-            </geometry>
-        </collision>
-        <xacro:inertial_cylinder mass="0.1" length="0.04" radius="0.05">
-            <origin xyz="0 0 0" rpy="0 0 0"/>
-        </xacro:inertial_cylinder>
     </link>
     <!-- RIGHT WHEEL LINK -->
-    <joint name="right_wheel_joint" type="continuous">
+        <joint name="right_wheel_joint" type="continuous">
         <parent link="base_link"/>
         <child link="right_wheel"/>
-        <origin xyz="0 -0.175 0" rpy="${pi/2} 0 0" />
+        <origin xyz="0 -0.080 0" rpy="${pi/2} 0 0" />
         <axis xyz="0 0 -1"/>
     </joint>
@@ -74,38 +56,8 @@
         <visual>
             <geometry>
-                <cylinder radius="0.05" length="0.04"/>
+                <cylinder radius="0.033" length="0.027"/>
             </geometry>
             <material name="blue"/>
         </visual>
-        <collision>
-            <geometry>
-                <cylinder radius="0.05" length="0.04"/>
-            </geometry>
-        </collision>
-        <xacro:inertial_cylinder mass="0.1" length="0.04" radius="0.05">
-            <origin xyz="0 0 0" rpy="0 0 0"/>
-        </xacro:inertial_cylinder>
-    </link>
-    <!-- CASTER WHEEL LINK -->
-    <joint name="caster_wheel_joint" type="fixed">
-        <parent link="chassis"/>
-        <child link="caster_wheel"/>
-        <origin xyz="0.24 0 0"/>
-    </joint>
-    <link name="caster_wheel">
-        <visual>
-            <geometry>
-                <sphere radius="0.05"/>
-            </geometry>
-            <material name="black"/>
-        </visual>
-        <collision>
-            <geometry>
-                <sphere radius="0.05"/>
-            </geometry>
-        </collision>
-        <xacro:inertial_sphere mass="0.1" radius="0.05">
-            <origin xyz="0 0 0" rpy="0 0 0"/>
-        </xacro:inertial_sphere>
     </link>
 </robot>

Commit message: added collision tags to the urdf

File: humble/workspace/src/my_bot/description/robot_core.xacro (robot description, xacro)
@@ -30,4 +30,10 @@
             <material name="white"/>
         </visual>
+        <collision>
+            <origin xyz="0.1025 0 0.0425"/>
+            <geometry>
+                <box size="0.205 0.125 0.085"/>
+            </geometry>
+        </collision>
     </link>
     <!-- LEFT WHEEL LINK -->
@@ -45,7 +51,12 @@
             <material name="blue"/>
         </visual>
+        <collision>
+            <geometry>
+                <cylinder radius="0.033" length="0.027"/>
+            </geometry>
+        </collision>
     </link>
     <!-- RIGHT WHEEL LINK -->
-        <joint name="right_wheel_joint" type="continuous">
+    <joint name="right_wheel_joint" type="continuous">
         <parent link="base_link"/>
         <child link="right_wheel"/>
@@ -60,4 +71,28 @@
             <material name="blue"/>
         </visual>
+        <collision>
+            <geometry>
+                <cylinder radius="0.033" length="0.027"/>
+            </geometry>
+        </collision>
+    </link>
+    <!-- CASTOR WHEEL LINK -->
+    <joint name="castor_wheel_joint" type="fixed">
+        <parent link="chassis"/>
+        <child link="castor_wheel"/>
+        <origin xyz="0.165 0 0"/>
+    </joint>
+    <link name="castor_wheel">
+        <visual>
+            <geometry>
+                <sphere radius="0.033" />
+            </geometry>
+            <material name="black"/>
+        </visual>
+        <collision>
+            <geometry>
+                <sphere radius="0.033" />
+            </geometry>
+        </collision>
     </link>
 </robot>

Commit message: add inertia macro file and update robot desciption with inertia values

File: humble/workspace/src/my_bot/description/robot_core.xacro (robot description, xacro)
@@ -1,4 +1,5 @@
 <?xml version="1.0"?>
 <robot xmlns:xacro="http://www.ros.org/wiki/xacro" >
+    <xacro:include filename="inertial_macros.xacro" />
     <material name="white">
         <color rgba="1 1 1 1" />
@@ -36,4 +37,7 @@
             </geometry>
         </collision>
+        <xacro:inertial_box mass = "0.5" x = "0.205" y = "0.125" z = "0.085">
+            <origin xyz="0.1025 0 0.0425" rpy = "0 0 0"/>
+        </xacro:inertial_box>
     </link>
     <!-- LEFT WHEEL LINK -->
@@ -56,4 +60,7 @@
             </geometry>
         </collision>
+        <xacro:inertial_cylinder mass = "0.035" length = "0.027" radius = "0.033">
+            <origin xyz="0 0 0" rpy = "0 0 0"/>
+        </xacro:inertial_cylinder>
     </link>
     <!-- RIGHT WHEEL LINK -->
@@ -76,4 +83,7 @@
             </geometry>
         </collision>
+        <xacro:inertial_cylinder mass = "0.035" length = "0.027" radius = "0.033">
+            <origin xyz="0 0 0" rpy = "0 0 0"/>
+        </xacro:inertial_cylinder>
     </link>
     <!-- CASTOR WHEEL LINK -->
@@ -95,4 +105,7 @@
             </geometry>
         </collision>
+        <xacro:inertial_sphere mass = "0.030" radius = "0.033">
+            <origin xyz="0 0 0" rpy = "0 0 0"/>
+        </xacro:inertial_sphere>
     </link>
 </robot>

Commit message: add a launch file to start rsp and gazebo, spawn robot in gazebo, add rviz config

File: humble/workspace/src/my_bot/description/robot_core.xacro (robot description, xacro)
@@ -41,4 +41,7 @@
         </xacro:inertial_box>
     </link>
+    <gazebo reference="chassis">
+        <material>Gazebo/White</material>
+    </gazebo>
     <!-- LEFT WHEEL LINK -->
     <joint name="left_wheel_joint" type="continuous">
@@ -64,4 +67,7 @@
         </xacro:inertial_cylinder>
     </link>
+    <gazebo reference="left_wheel">
+        <material>Gazebo/Blue</material>
+    </gazebo>
     <!-- RIGHT WHEEL LINK -->
     <joint name="right_wheel_joint" type="continuous">
@@ -87,4 +93,7 @@
         </xacro:inertial_cylinder>
     </link>
+    <gazebo reference="right_wheel">
+        <material>Gazebo/Blue</material>
+    </gazebo>
     <!-- CASTOR WHEEL LINK -->
     <joint name="castor_wheel_joint" type="fixed">
@@ -109,3 +118,8 @@
         </xacro:inertial_sphere>
     </link>
+    <gazebo reference="castor_wheel">
+        <material>Gazebo/Black</material>
+        <mu1 value="0.00001"/>
+        <mu2 value="0.00001"/>
+    </gazebo>
 </robot>

Commit message: updated box dimention to match new chassis

File: humble/workspace/src/my_bot/description/robot_core.xacro (robot description, xacro)
@@ -21,22 +21,22 @@
         <parent link="base_link"/>
         <child link="chassis"/>
-        <origin xyz="-0.055 0 0"/>
+        <origin xyz="-0.125 0 0"/>
     </joint>
     <link name="chassis">
         <visual>
-            <origin xyz="0.1025 0 0.0425"/>
+            <origin xyz="0.185 0 0.07"/>
             <geometry>
-                <box size="0.205 0.125 0.085"/>
+                <box size="0.370 0.230 0.140"/>
             </geometry>
             <material name="white"/>
         </visual>
         <collision>
-            <origin xyz="0.1025 0 0.0425"/>
+            <origin xyz="0.185 0 0.07"/>
             <geometry>
-                <box size="0.205 0.125 0.085"/>
+                <box size="0.370 0.230 0.140"/>
             </geometry>
         </collision>
-        <xacro:inertial_box mass = "0.5" x = "0.205" y = "0.125" z = "0.085">
-            <origin xyz="0.1025 0 0.0425" rpy = "0 0 0"/>
+        <xacro:inertial_box mass = "1.4" x = "0.370" y = "0.230" z = "0.140">
+            <origin xyz="0.185 0 0.07" rpy = "0 0 0"/>
         </xacro:inertial_box>
     </link>
@@ -48,5 +48,5 @@
         <parent link="base_link"/>
         <child link="left_wheel"/>
-        <origin xyz="0 0.080 0" rpy="-${pi/2} 0 0" />
+        <origin xyz="0 0.120 0" rpy="-${pi/2} 0 0" />
         <axis xyz="0 0 1"/>
     </joint>
@@ -74,5 +74,5 @@
         <parent link="base_link"/>
         <child link="right_wheel"/>
-        <origin xyz="0 -0.080 0" rpy="${pi/2} 0 0" />
+        <origin xyz="0 -0.120 0" rpy="${pi/2} 0 0" />
         <axis xyz="0 0 -1"/>
     </joint>
@@ -100,5 +100,5 @@
         <parent link="chassis"/>
         <child link="castor_wheel"/>
-        <origin xyz="0.165 0 0"/>
+        <origin xyz="0.270 0 0"/>
     </joint>
     <link name="castor_wheel">
