Commit message: added laser scanner in gazebo

File: humble/workspace/src/my_bot/description/gazebo_control.xacro (robot description, xacro)
@@ -6,5 +6,5 @@
             <left_joint>left_wheel_joint</left_joint>
             <right_joint>right_wheel_joint</right_joint>
-            <wheel_separation>0.16</wheel_separation>
+            <wheel_separation>0.240</wheel_separation>
             <wheel_diameter>0.033</wheel_diameter>
             <!-- Limits -->

File: humble/workspace/src/my_bot/description/robot_core.xacro (robot description, xacro)
@@ -13,4 +13,7 @@
     <material name="black">
         <color rgba="0 0 0 1"/>
+    </material>
+    <material name="red">
+        <color rgba="1 0 0 1"/>
     </material>
     <!-- BASE LINK -->
